Commit message: added lidar sensor and instructions in readme.md

File: urdf/simple_robot.urdf (robot description, URDF)
Before this commit: robot simple_robot, 3 links, 2 joints
Links:
- added link lidar_link, mass 0.1; collision cylinder length=0.05 radius=0.05; visual cylinder length=0.05 radius=0.05
Joints:
- added joint lidar_joint: type fixed, parent base_link, child lidar_link, origin xyz=0.15 0 0.15 rpy=0 0 0
